Commit message: Modification with Slash being missing, as well as </link>

File: description/robot_core.xacro (robot description, xacro)
@@ -2,17 +2,18 @@
 <robot xmlns:xacro="http://www.ros.org/wiki/xacro" >
     <material name="white">
-        <color rgba= "1 1 1 1">
+        <color rgba= "1 1 1 1"/>
     </material>
     <material name="orange">
-        <color rgba= "1 0.3 0.1 1">
+        <color rgba= "1 0.3 0.1 1"/>
     </material>
     <material name="blue">
-        <color rgba= "0.2 0.2 1 1">
+        <color rgba= "0.2 0.2 1 1"/>
     </material>
     <material name="black">
-        <color rgba= "0 0 0 1">
+        <color rgba= "0 0 0 1"/>
     </material>
     <!-- Apparenly its a standard for ROS2 to have the first link as the "Base Link" -->
     <link name="base_link">
+    </link>
     <joint name="chassis_joint" type="fixed">
         <parent link="base_link"/>
@@ -28,3 +29,4 @@
             <material name="white"/>
         </visual>
+    </link>
 </robot>

Commit message: finished code

File: description/robot_core.xacro (robot description, xacro)
@@ -1,4 +1,5 @@
 <?xml version="1.0"?>
 <robot xmlns:xacro="http://www.ros.org/wiki/xacro" >
+    <xacro:include filename="inertial_macros.xacro"/>
     <material name="white">
         <color rgba="1 1 1 1"/>
@@ -13,7 +14,8 @@
         <color rgba="0 0 0 1"/>
     </material>
-    <!-- Apparenly its a standard for ROS2 to have the first link as the "Base Link" -->
-    <link name="base_link">
+    <!-- BASE LINK -->
+    <link name="base_link"> <!-- Apparenly its a standard for ROS2 to have the first link as the "Base Link" -->
     </link>
+    <!-- CHASSIS LINK -->
     <joint name="chassis_joint" type="fixed">
         <parent link="base_link"/>
@@ -24,9 +26,86 @@
         <visual>
             <origin xyz="0.15 0 0.075"/>
+                <geometry>
+                    <box size="0.3 0.3 0.15"/> <!-- Values in meters -->
+            </geometry>
+            <material name="white"/>
+        </visual>
+        <collision>
+            <origin xyz="0.15 0 0.075"/>
             <geometry>
                 <box size="0.3 0.3 0.15"/> <!-- Values in meters -->
             </geometry>
-            <material name="white"/>
+        </collision>
+        <xacro:inertial_box mass="0.5" x="0.3" y="0.3" z="0.15">
+            <origin xyz="0.15 0 0.75" rpy="0 0 0"/>
+        </xacro:inertial_box>
+    </link>
+    <!-- LEFT WHEEL LINK -->
+    <joint name="left_wheel_joint" type="continuous">
+        <parent link="base_link"/>
+        <child link="left_wheel"/>
+        <origin xyz="0 0.175 0" rpy="-${pi/2} 0 0"/> <!-- Roll Pitch Yaw (rpy) and origin is slightly to the left so its not in the center of the chassis-->
+        <axis xyz="0 0 1"/> <!-- Specify an axis of rotation, when we have positive motion in the wheels, we need to be positive around z,  anticlockwise for robot to move forward-->
+    </joint>
+    <link name="left_wheel">
+        <visual>
+            <geometry>
+                <cylinder radius="0.05" length="0.04"/>
+            </geometry>
+            <material name="blue"/>
         </visual>
+        <collision>
+            <geometry>
+                <cylinder radius="0.05" length="0.04"/>
+            </geometry>
+        </collision>
+        <xacro:inertial_cylinder mass="0.1" length="0.04" radius="0.05">
+            <origin xyz="0 0 0" rpy="0 0 0"/>
+        </xacro:inertial_cylinder>
+    </link>
+     <!-- RIGHT WHEEL LINK -->
+    <joint name="right_wheel_joint" type="continuous">
+        <parent link="base_link"/>
+        <child link="right_wheel"/>
+        <origin xyz="0 -0.175 0" rpy="${pi/2} 0 0"/> <!-- Roll Pitch Yaw (rpy) and origin is slightly to the left so its not in the center of the chassis-->
+        <axis xyz="0 0 -1"/> <!-- Specify an axis of rotation, when we have positive motion in the wheels, we need to be positive around z,  anticlockwise for robot to move forward-->
+    </joint>
+    <link name="right_wheel">
+        <visual>
+            <geometry>
+                <cylinder radius="0.05" length="0.04"/>
+            </geometry>
+            <material name="blue"/>
+        </visual>
+        <collision>
+            <geometry>
+                <cylinder radius="0.05" length="0.04"/>
+            </geometry>
+        </collision>
+        <xacro:inertial_cylinder mass="0.1" length="0.04" radius="0.05">
+            <origin xyz="0 0 0" rpy="0 0 0"/>
+        </xacro:inertial_cylinder>
+    </link>
+    <!-- CASTER WHEEL LINK -->
+    <joint name="caster_wheel_joint" type="fixed">
+        <parent link="chassis"/>
+        <child link="caster_wheel"/>
+        <origin xyz="0.24 0 0"/>
+    </joint>
+    <link name="caster_wheel">
+        <visual>
+            <geometry>
+                <sphere radius="0.05"/>
+            </geometry>
+            <material name="black"/>
+        </visual>
+       <collision>
+            <geometry>
+                <sphere radius="0.05"/>
+            </geometry>
+        </collision>
+        <xacro:inertial_sphere mass="0.1" radius="0.05">
+            <origin xyz="0 0 0" rpy ="0 0 0"/>
+        </xacro:inertial_sphere>
     </link>
 </robot>
